Commit message: fix biotac model

File: sr_description/hand/xacro/finger/distal/distal.urdf.xacro (robot description, xacro)
@@ -130,5 +130,5 @@
         <parent link="${prefix}${link_prefix}distal" />
         <child link="${prefix}${link_prefix}tip" />
-        <origin xyz="0 0 0.026" rpy="0 0 0" />
+        <origin xyz="0 0 0.034" rpy="0 0 0" />
       </joint>
     </xacro:unless>

File: sr_description/hand/xacro/thumb/thdistal.urdf.xacro (robot description, xacro)
@@ -18,5 +18,5 @@
   params="muscle bio bt_sp ubi eli prefix parent">
     <xacro:if value="${bio}">
-      <!--    BIOTAC -->
+      <!-- BIOTAC -->
       <link name="${prefix}thdistal_J1_dummy">
         <inertial>
@@ -112,7 +112,5 @@
         <parent link="${prefix}thdistal_J1_dummy" />
         <child link="${prefix}thtip" />
-        <origin xyz="0.0 0.004 ${0.032}"
-        rpy="0 0 0" />
-        <!-- approximated only FIXME -->
+        <origin xyz="0.0 0.0036" rpy="0 0 0" />
       </joint>
     </xacro:if>
@@ -127,5 +125,5 @@
         </inertial>
         <visual>
-          <origin xyz="0 0 0" rpy="0 0 0" />
+          <origin xyz="0 0 0.0022" rpy="0 0 0" />
           <geometry name="${prefix}thdistal_visual">
             <xacro:if value="${eli}">
@@ -140,15 +138,15 @@
                       scale="0.001 0.001 0.001" />
               </xacro:if>
-	      <xacro:unless value="${ubi}">
-		<xacro:if value="${bt_sp}">
-		  <!-- bt sp distal  -->
-		  <mesh filename="package://sr_description/hand/model/biotacs/sp.dae" />
-		</xacro:if>
-		<xacro:unless value="${bt_sp}">
-		  <!-- Standard distal  -->
-                  <mesh filename="package://sr_description/hand/model/TH1_z.dae"
-			scale="0.001 0.001 0.001" />
-		</xacro:unless>
-	      </xacro:unless>
+	          <xacro:unless value="${ubi}">
+		        <xacro:if value="${bt_sp}">
+		          <!-- bt sp distal  -->
+		          <mesh filename="package://sr_description/hand/model/biotacs/sp.dae" />
+		        </xacro:if>
+	        	<xacro:unless value="${bt_sp}">
+		          <!-- Standard distal  -->
+              <mesh filename="package://sr_description/hand/model/TH1_z.dae"
+			                scale="0.001 0.001 0.001" />
+		        </xacro:unless>
+	          </xacro:unless>
             </xacro:unless>
           </geometry>
@@ -158,5 +156,5 @@
         </visual>
         <collision>
-          <origin xyz="0 0 0" rpy="0 0 0" />
+          <origin xyz="0 0 0.0022" rpy="0 0 0" />
           <geometry name="${prefix}thmiddle_collision_geom">
             <xacro:if value="${eli}">
@@ -172,13 +170,13 @@
               </xacro:if>
               <xacro:unless value="${ubi}">
-		<xacro:if value="${bt_sp}">
-		  <!-- bt sp distal  -->
-                  <mesh filename="package://sr_description/hand/model/biotacs/sp.dae" />
-		</xacro:if>
-		<xacro:unless value="${bt_sp}">
+		            <xacro:if value="${bt_sp}">
+		              <!-- bt sp distal  -->
+                    <mesh filename="package://sr_description/hand/model/biotacs/sp.dae" />
+	            	</xacro:if>
+		            <xacro:unless value="${bt_sp}">
                   <!-- Standard distal  -->
                   <mesh filename="package://sr_description/hand/model/TH1_z.dae"
-			scale="0.001 0.001 0.001" />
-		</xacro:unless>
+			            scale="0.001 0.001 0.001" />
+		            </xacro:unless>
               </xacro:unless>
             </xacro:unless>
@@ -210,5 +208,5 @@
         <parent link="${prefix}thdistal" />
         <child link="${prefix}thtip" />
-        <origin xyz="0 0 0.0275" rpy="0 0 0" />
+        <origin xyz="0 0 0.0362" rpy="0 0 0" />
       </joint>
       <xacro:thdistal_gazebo prefix="${prefix}" />

Commit message: add if unless parameter

File: sr_description/hand/xacro/finger/distal/distal.urdf.xacro (robot description, xacro)
@@ -130,5 +130,10 @@
         <parent link="${prefix}${link_prefix}distal" />
         <child link="${prefix}${link_prefix}tip" />
-        <origin xyz="0 0 0.034" rpy="0 0 0" />
+        <xacro:if value="${bt_sp}">
+          <origin xyz="0 0 0.034" rpy="0 0 0" />
+		    </xacro:if>
+		    <xacro:unless value="${bt_sp}">
+          <origin xyz="0 0 0.026" rpy="0 0 0" />
+		    </xacro:unless>
       </joint>
     </xacro:unless>

File: sr_description/hand/xacro/thumb/thdistal.urdf.xacro (robot description, xacro)
@@ -125,5 +125,10 @@
         </inertial>
         <visual>
-          <origin xyz="0 0 0.0022" rpy="0 0 0" />
+          <xacro:if value="${bt_sp}">
+            <origin xyz="0 0 0.0022" rpy="0 0 0" />
+		      </xacro:if>
+		      <xacro:unless value="${bt_sp}">
+            <origin xyz="0 0 0" rpy="0 0 0" />
+		      </xacro:unless>
           <geometry name="${prefix}thdistal_visual">
             <xacro:if value="${eli}">
@@ -156,5 +161,10 @@
         </visual>
         <collision>
-          <origin xyz="0 0 0.0022" rpy="0 0 0" />
+          <xacro:if value="${bt_sp}">
+            <origin xyz="0 0 0.0022" rpy="0 0 0" />
+		      </xacro:if>
+		      <xacro:unless value="${bt_sp}">
+            <origin xyz="0 0 0" rpy="0 0 0" />
+		      </xacro:unless>
           <geometry name="${prefix}thmiddle_collision_geom">
             <xacro:if value="${eli}">
@@ -208,5 +218,10 @@
         <parent link="${prefix}thdistal" />
         <child link="${prefix}thtip" />
-        <origin xyz="0 0 0.0362" rpy="0 0 0" />
+        <xacro:if value="${bt_sp}">
+          <origin xyz="0 0 0.034" rpy="0 0 0" />
+		    </xacro:if>
+		    <xacro:unless value="${bt_sp}">
+          <origin xyz="0 0 0.026" rpy="0 0 0" />
+		    </xacro:unless>
       </joint>
       <xacro:thdistal_gazebo prefix="${prefix}" />
